File: BoardyMcBoardFace/BoardyMcBoardFace.sch (KiCad schematic (older format))
At the start: 40 parts

Commit message: wip
Parts:
- removed D? (x3): LED, symbol Device:LED
- removed J?: Conn_01x06_Male, symbol Connector:Conn_01x06_Male
- removed J?: Conn_01x05_Male, symbol Connector:Conn_01x05_Male
- removed R? (x3): 100, symbol Device:R
- removed U?: NRF24L01, Package_DFN_QFN:QFN-20-1EP_4x4mm_P0.5mm_EP2.5x2.5mm, symbol RF:NRF24L01
- removed U? (x2): OPAMP, symbol pspice:OPAMP
- added C10, C11, C9: 10n, Capacitor_SMD:C_0402_1005Metric, symbol Device:C
- added C12: 33n, Capacitor_SMD:C_0402_1005Metric, symbol Device:C
- added C15: 1p5, Capacitor_SMD:C_0402_1005Metric, symbol Device:C
- added C16: 1p, Capacitor_SMD:C_0402_1005Metric, symbol Device:C
- added C17: 2n2, Capacitor_SMD:C_0402_1005Metric, symbol Device:C
- added C18: 4p7, Capacitor_SMD:C_0402_1005Metric, symbol Device:C
- added C3: 100n, Capacitor_SMD:C_0402_1005Metric, symbol Device:C
- added C8: 10u, Capacitor_SMD:C_0603_1608Metric, symbol Device:C
- added C? (x2): 22u, symbol Device:C
- added C? (x2): 12p, Capacitor_SMD:C_0402_1005Metric, symbol Device:C
- added D? (x3): LED, symbol Device:LED
- added J2: SMA, Connector_Coaxial:SMA_Samtec_SMA-J-P-X-ST-EM1_EdgeMount, symbol Connector:Conn_Coaxial
- added J3: ARM 10pin, Connector_PinHeader_1.27mm:PinHeader_2x05_P1.27mm_Vertical, symbol Connector_Generic:Conn_02x05_Odd_Even
- added L1: 3n9, Inductor_SMD:L_0402_1005Metric, symbol Device:L
- added L2: 8n2, Inductor_SMD:L_0402_1005Metric, symbol Device:L
- added L3: 2n7, Inductor_SMD:L_0402_1005Metric, symbol Device:L
- added R4: 22k, Resistor_SMD:R_0402_1005Metric, symbol Device:R
- added R? (x3): 100, symbol Device:R
- added R?: 1M, Resistor_SMD:R_0402_1005Metric, symbol Device:R
- added U4: nRF24L01P, Package_DFN_QFN:QFN-20-1EP_4x4mm_P0.5mm_EP2.5x2.5mm, symbol RF:nRF24L01P
- added Y?: 16MHz, Crystal:Crystal_SMD_3225-4Pin_3.2x2.5mm, symbol Device:Crystal_GND24_Small
Connections:
- net labels added: +3V3, NRF_AN1, NRF_AN2, NRF_ANT1, NRF_ANT2, NRF_VDD_PA, NRF_XC1, NRF_XC2, RADIO_CE, USB_LED
- wire segments 125 -> 222
- no-connect marks 3 -> 7
Other:
- note added: "Antenna Impedance Matching and SMA Connector"
- note added: "Load caps: C = 2 * (Cload - Cstray)"
- note added: "Mr.Clean"
- note added: "NRF24 Transceiver"
- note added: "NRST cap not strictly necessary\nbut protects against parasitic resets."
- note added: "Passive antenna."
- note added: "Route as 50 Ohm controlled impedance traces.\nFollow datasheet regarding layout."
- note added: "SWD Connector"
- note added: "Transceiver Crystal"
- note removed: "STLINK Connector\n"
- moved on the sheet: C?, D?, FB?, J?, R?, SW?, U?, Y?

Commit message: wip
Parts:
- added C12, C13, C2, C3: 10p, symbol Device:C
- added C15, C16, C6, C7: 10n, symbol Device:C
- added D1, D10, D11, D19, D2, D20, D7, D8: LED, symbol Device:LED
- added D12, D17, D18, D21, D22, D23, D24, D25, D26, D27, D28, D9: WS2812B, LED_SMD:LED_WS2812B_PLCC4_5.0x5.0mm_P3.2mm, symbol LED:WS2812B
- added D13, D14, D3, D4: LD271, LED_THT:LED_D5.0mm_IRGrey, symbol LED:LD271
- added D15, D16, D5, D6: D_Photo, symbol Device:D_Photo
- added J1: Conn_01x14_Female, symbol Connector:Conn_01x14_Female
- added J?: Conn_01x04, symbol Connector_Generic:Conn_01x04
- added R1, R13, R14, R15, R16, R2, R23, R24: 1k, symbol Device:R
- added R10, R11, R19, R20, R21, R22, R7, R8: 10k, symbol Device:R
- added R17, R18, R5, R6: 100, symbol Device:R
- added RV1, RV2, RV3, RV4: R_POT 10k, symbol Device:R_POT
- added SW?: SW_DPDT_x2, symbol Switch:SW_DPDT_x2
- added TP1, TP2, TP3, TP4, TP5: TestPoint, symbol Connector:TestPoint
- added TP6, TP7, TP8, TP9: TestPoint_Flag, symbol Connector:TestPoint_Flag
- added U2, U3, U5, U6: LM393, symbol Comparator:LM393
- gave numbers to parts that had none: 41
- renumbered C12 to C20, C8 to C21, C17 to C22, C9 to C23, C18 to C24, C10 to C25, C15 to C26, C16 to C27, C11 to C29, C3 to C33, J3 to J4, L2 to L1, L1 to L2, R4 to R25, U4 to U8
Connections:
- net labels added: BALLDETECT_1, BALLDETECT_2, BALLDETECT_3, BALLDETECT_4, PB11, PIXEL_MISO, PIXEL_MOSI, PIXEL_OFFBOARD_OUT, PIXEL_OUT, PIXEL_SCK, PIXEl_MISO
- net labels removed: FAULT_LED, NRF_AN1, NRF_AN2, PA8, PB12, PB13, PB14, PB15, PC14, PC15, PIXEL_1, PIXEL_2
- wire segments 222 -> 399
- no-connect marks 7 -> 6
Other:
- note added: "Ball Detectors\n"
- note added: "Breakout"
- note added: "Flip switch to connect node 2 to 3 when no offboard\nneopixels are connected. Otherwise connect node 2\nto 1 to route through the connector"
- note added: "If the neopixels need to be daisy-chained\noffboard, they need to be disconected \nfrom the microcontroller and connected\n to the offboard connector\n"
- note added: "Neopixels\n"
- note added: "PIXEL_SCK is tied to the neopixel SPI MOSI. This signal\nisn't reallyuseful if its always tied up in the SPI peripheral.\nBut its broken out here just incase there is a way to free it."
- note added: "Spec the 128kb ram\nand 20kb sram\n"
- note added: "Test Points\n"
- moved on the sheet: C30, C32, C33, R27, U4, Y2

Commit message: add footprints
Parts:
- removed R3: 10k, symbol Device:R
- removed SW1, SW2: SW_SPDT, symbol Switch:SW_SPDT
- added C5: 0.1u, Capacitor_SMD:C_0201_0603Metric, symbol Device:C
- added R23: 120, Resistor_SMD:R_0402_1005Metric, symbol Device:R
- added SW1: SW_Push, Button_Switch_SMD:SW_Push_SPST_NO_Alps_SKRK, symbol Switch:SW_Push
- added SW2: SW_DIP_x02, Button_Switch_THT:SW_DIP_SPSTx02_Slide_9.78x7.26mm_W7.62mm_P2.54mm, symbol Switch:SW_DIP_x02
- C1, C2, C3: footprint (none) -> Capacitor_SMD:C_0402_1005Metric
- C10: renamed from C9; footprint (none) -> Capacitor_SMD:C_0603_1608Metric
- C11: renamed from C10; footprint (none) -> Capacitor_SMD:C_0603_1608Metric
- C12: renamed from C11; footprint (none) -> Capacitor_SMD:C_0603_1608Metric
- C13: renamed from C12; footprint (none) -> Capacitor_SMD:C_0402_1005Metric
- C14: renamed from C13; footprint (none) -> Capacitor_SMD:C_0402_1005Metric
- C15: renamed from C14; footprint (none) -> Capacitor_SMD:C_0603_1608Metric
- C16: renamed from C15; footprint (none) -> Capacitor_SMD:C_0402_1005Metric
- C17: renamed from C16; footprint (none) -> Capacitor_SMD:C_0402_1005Metric
- C18: renamed from C17; footprint (none) -> Capacitor_SMD:C_0603_1608Metric
- C19: renamed from C18; footprint (none) -> Capacitor_SMD:C_0603_1608Metric
- C20: renamed from C19; footprint (none) -> Capacitor_SMD:C_0603_1608Metric
- C29: renamed from C28; footprint (none) -> Capacitor_SMD:C_0805_2012Metric
- C32: renamed from C31; footprint (none) -> Capacitor_SMD:C_0805_2012Metric
- C4: footprint (none) -> Capacitor_SMD:C_0201_0603Metric
- C6: renamed from C5; footprint (none) -> Capacitor_SMD:C_0402_1005Metric
- C7: renamed from C6; footprint (none) -> Capacitor_SMD:C_0402_1005Metric
- C8: renamed from C7; footprint (none) -> Capacitor_SMD:C_0402_1005Metric
- C9: renamed from C8; footprint (none) -> Capacitor_SMD:C_0603_1608Metric
- D1, D10, D11, D19, D2, D20, D31, D32, D33, D7, D8: footprint (none) -> LED_SMD:LED_0402_1005Metric
- D15, D16, D5, D6: footprint (none) -> Diode_THT:D_5KPW_P7.62mm_Vertical_AnodeUp
- D29, D30: footprint (none) -> Diode_SMD:D_0805_2012Metric
- FB1: footprint (none) -> Inductor_SMD:L_0603_1608Metric
- J1: footprint (none) -> Connector_PinSocket_2.54mm:PinSocket_1x14_P2.54mm_Vertical
- J2: renamed from J?; footprint (none) -> Connector:FanPinHeader_1x04_P2.54mm_Vertical
- J4: renamed from J3; footprint (none) -> Connector:FanPinHeader_1x04_P2.54mm_Vertical
- J6: renamed from J5; footprint (none) -> Connector_USB:USB_Micro-B_Wuerth_629105150521
- R1, R2, R26, R28, R29, R30: footprint (none) -> Resistor_SMD:R_0402_1005Metric
- R10: renamed from R12; footprint (none) -> Resistor_SMD:R_0402_1005Metric
- R11: renamed from R13; footprint (none) -> Resistor_SMD:R_0402_1005Metric
- R12: renamed from R14; footprint (none) -> Resistor_SMD:R_0402_1005Metric
- R13: renamed from R15; footprint (none) -> Resistor_SMD:R_0402_1005Metric
- R14: renamed from R16; footprint (none) -> Resistor_SMD:R_0402_1005Metric
- R15: renamed from R17; footprint (none) -> Resistor_SMD:R_0402_1005Metric
- R16: renamed from R18; footprint (none) -> Resistor_SMD:R_0402_1005Metric
- R17: renamed from R19; footprint (none) -> Resistor_SMD:R_0402_1005Metric
- R18: renamed from R20; footprint (none) -> Resistor_SMD:R_0402_1005Metric
- R19: renamed from R21; footprint (none) -> Resistor_SMD:R_0402_1005Metric
- R20: renamed from R22; footprint (none) -> Resistor_SMD:R_0402_1005Metric
- R21: renamed from R23; footprint (none) -> Resistor_SMD:R_0402_1005Metric
- R22: renamed from R24; footprint (none) -> Resistor_SMD:R_0402_1005Metric
- R24: renamed from R4; footprint (none) -> Resistor_SMD:R_0402_1005Metric
- R3: renamed from R5; footprint (none) -> Resistor_SMD:R_0402_1005Metric
- R4: renamed from R6; footprint (none) -> Resistor_SMD:R_0402_1005Metric
- R5: renamed from R7; footprint (none) -> Resistor_SMD:R_0402_1005Metric
- R6: renamed from R8; footprint (none) -> Resistor_SMD:R_0402_1005Metric
- R7: renamed from R9; footprint (none) -> Resistor_SMD:R_0402_1005Metric
- R8: renamed from R10; footprint (none) -> Resistor_SMD:R_0402_1005Metric
- R9: renamed from R11; footprint (none) -> Resistor_SMD:R_0402_1005Metric
- RV1, RV2, RV3, RV4: footprint (none) -> ExtraStuff:BOURNS-3362P_pot
- SW3: renamed from SW?; footprint (none) -> Button_Switch_THT:SW_E-Switch_EG1271_DPDT
- TP1, TP2, TP3, TP4, TP5: footprint (none) -> TestPoint:TestPoint_Plated_Hole_D2.0mm
- TP6, TP7, TP8, TP9: footprint (none) -> TestPoint:TestPoint_Pad_1.5x1.5mm
- U2, U3, U5, U6: footprint (none) -> Package_SO:SOIC-8_3.9x4.9mm_P1.27mm
- Y1: footprint (none) -> Crystal:Crystal_SMD_3225-4Pin_3.2x2.5mm
- renumbered C20 to C21, C21 to C22, C22 to C23, C23 to C24, C24 to C25, C25 to C26, C26 to C27, C27 to C28, C29 to C30, C30 to C31, C32 to C33, C33 to C34, J2 to J3, J4 to J5
Connections:
- net PIXEl_MISO is gone; now on net PIXEL_MISO: J2.2 (Pin_2)
- net +3V3: now also R24.2
- net BOOT: now also SW2.3
- net CAN_H: now also R23.1
- net CAN_L: now also SW2.1
- net GND: now also C5.2, SW1.1, SW2.2
- net NRST: now also C5.1, SW1.2
- new net: R23.2, SW2.4
Other:
- note added: "Enable switch to switch to boot mode 0\nDefault to boot mode 1"
- note added: "MainBoard"
- note added: "Optional CAN termination. Enable switch\n1-4 if this is the last node on the bus.\nDisable if connected to the CAN distribution\nboard."
- moved on the sheet: J1, R24
