File: SX1280_USB_Adapter/SX1280_USB_Adapter.kicad_pcb (KiCad board)
At the start: 2 copper layers, 14 parts, among them J2 Conn_01x07, J3 Conn_01x07, U1 AMS1117-3.3, U2 CH341a, Y1 12M

Commit message: schematic done
Parts:
- removed J2, J3: Conn_01x07, Connector_PinSocket_2.54mm:PinSocket_1x07_P2.54mm_Vertical
- removed RN1: 222, Resistor_SMD:R_Array_Convex_4x0603
- added D3: LED, LED_SMD:LED_0603_1608Metric, F.Cu at (176.3, 93.6)
- added D4: LED, LED_SMD:LED_0603_1608Metric, F.Cu at (176.3, 96.1)
- added J1: USB_A_PLUG, USB_PCB:USB_PCB, F.Cu at (149.6, 117.8)
- added R2: R330, Resistor_SMD:R_0402_1005Metric, F.Cu at (170.6, 116.4)
- added R3: R330, Resistor_SMD:R_0402_1005Metric, F.Cu at (170.6, 118.4)
- added R4: R330, Resistor_SMD:R_0402_1005Metric, F.Cu at (170.6, 120.4)
- added R5: 1k, Resistor_SMD:R_0402_1005Metric, F.Cu at (170.6, 122.4)
- added R6: R330, Resistor_SMD:R_0402_1005Metric, F.Cu at (170.6, 124.4)
- added TP1: TestPoint, TestPoint:TestPoint_Pad_1.0x1.0mm, F.Cu at (169.7, 88.6)
- added TP2: TestPoint, TestPoint:TestPoint_Pad_1.0x1.0mm, F.Cu at (169.7, 91.7)
- added TP3: TestPoint, TestPoint:TestPoint_Pad_1.0x1.0mm, F.Cu at (169.7, 94.7)
- added TP4: TestPoint, TestPoint:TestPoint_Pad_1.0x1.0mm, F.Cu at (169.7, 97.8)
- added TP5: TestPoint, TestPoint:TestPoint_Pad_1.0x1.0mm, F.Cu at (172.7, 88.6)
- added TP6: TestPoint, TestPoint:TestPoint_Pad_1.0x1.0mm, F.Cu at (172.7, 91.7)
- added TP7: TestPoint, TestPoint:TestPoint_Pad_1.0x1.0mm, F.Cu at (172.7, 94.7)
- added U3: SX1280, SX1280:E28-2G4M12S-SX1280, F.Cu at (155.8, 96.2)
- C1, C2, C4, C5: footprint Capacitor_SMD:C_0603_1608Metric -> Capacitor_SMD:C_0402_1005Metric
- C3: value 472 -> 47p2; footprint Capacitor_SMD:C_0603_1608Metric -> Capacitor_SMD:C_0402_1005Metric
- D1: value Power -> LED
- D2: value RUN -> LED
- R1: value 0R -> 0; footprint Resistor_SMD:R_0805_2012Metric -> Resistor_SMD:R_0402_1005Metric
- Y1: value 12M -> Crystal_GND24; footprint Crystal:Crystal_HC49-U_Vertical -> Crystal:Crystal_SMD_3225-4Pin_3.2x2.5mm
- moved U1 137.7 mm to (174.0, 109.3)
- moved Y1 137.1 mm to (181.2, 118.1)
- moved U2 135.0 mm to (162.7, 114.9)
- moved C1 133.8 mm to (173.5, 114.4)
- moved C2 133.5 mm to (173.5, 116.4)
- moved C3 133.2 mm to (173.5, 118.4)
- moved C4 132.9 mm to (173.5, 120.3)
- moved C5 132.6 mm to (173.5, 122.3)
- moved R1 125.4 mm to (170.6, 114.4)
- moved D1 117.8 mm to (176.3, 88.4)
- moved D2 117.8 mm to (176.3, 91.0)
Connections:
- C1 pad 1: Net-(U2-XI) -> /GND
- C1 pad 2: Earth -> Net-(U2-XI)
- C2 pad 1: /5V -> /GND
- C2 pad 2: Earth -> /5V
- C3 pad 1: Net-(U2-V3) -> /GND
- C3 pad 2: Earth -> Net-(U2-V3)
- C4 pad 1: Net-(U2-XO) -> /GND
- C4 pad 2: Earth -> Net-(U2-XO)
- C5 pad 1: /3V3 -> /GND
- C5 pad 2: Earth -> /3V3
- D1 pad 1: Earth -> /GND
- D2 pad 1: Net-(D2-K) -> /GND
- D2 pad 2: /3V3 -> Net-(D2-A)
- U1 pad 1: Earth -> /GND
- U2 pad 1: Net-(RN1D-R4.1) -> unconnected-(U2-~{ACT}-Pad1)
- U2 pad 12: Earth -> /GND
- U2 pad 23: /SDA -> unconnected-(U2-SDA-Pad23)
- U2 pad 27: Earth -> /GND
- U2 pad 5: /TXD -> unconnected-(U2-TXD/~{ERR/USERDEF}-Pad5)
- U2 pad 6: /RXD -> unconnected-(U2-RXD/PEMP/USERDEF-Pad6)
- Y1 pad 2: Net-(U2-XO) -> /GND
Other:
- board outline added: 45 x 19.6 mm

Commit message: update layout
Parts:
- added TP8: TestPoint, TestPoint:TestPoint_Pad_1.0x1.0mm, F.Cu at (113.3, 121.7)
- U3: moved to B.Cu
- moved D1 68.4 mm to (110.5, 106.9), turned to 90 degrees
- moved C2 64.9 mm to (108.6, 113.8), turned to -90 degrees
- moved D4 63.7 mm to (113.5, 106.9), turned to 90 degrees
- moved TP2 61.8 mm to (115.7, 121.7)
- moved C5 61.3 mm to (112.3, 118.1)
- moved R1 60.4 mm to (110.2, 118.1), turned to 180 degrees
- moved U1 60.4 mm to (113.8, 113.8)
- moved Y1 59.9 mm to (122.5, 106.4), turned to 180 degrees
- moved R2 59.3 mm to (112.0, 107.4), turned to 90 degrees
- moved TP6 58.9 mm to (122.0, 121.6)
- moved TP5 56.8 mm to (126.5, 121.6)
- moved R3 56.6 mm to (115.0, 107.4), turned to 90 degrees
- moved C4 55.7 mm to (119.5, 106.5), turned to -90 degrees
- moved TP7 55.4 mm to (124.3, 121.6)
- moved J1 53.0 mm to (96.7, 114.0), turned to -90 degrees
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Other:
- board text added: "3v3"
- board text added: "5v"
- board text added: "The Bots"
- board text added: "ck"
- board text added: "cs"
- board text added: "gnd"
- board text added: "mi"
- board text added: "mo"

Commit message: layout finished
Parts:
- removed R1: 0, Resistor_SMD:R_0402_1005Metric
- R5: moved to B.Cu
- moved TP2 15.7 mm to (115.0, 106.0)
- moved TP8 15.7 mm to (113.0, 106.0)
- moved D1 14.2 mm to (112.5, 121.0)
- moved D4 14.1 mm to (114.5, 121.0)
- moved R2 13.9 mm to (111.0, 121.2)
- moved R3 13.4 mm to (115.8, 120.8)
- moved C5 7.81 mm to (119.0, 114.0), turned to 90 degrees
- moved R4 2.02 mm to (140.5, 106.2), turned to 90 degrees
- moved R5 1.80 mm to (129.0, 105.0), turned to 180 degrees
- moved D2 1.33 mm to (139.0, 106.2)
- moved TP3 1.11 mm to (136.0, 122.0)
- moved R6 0.97 mm to (135.5, 106.2)
- moved TP1 0.89 mm to (138.0, 122.0)
- moved D3 0.53 mm to (137.0, 106.2)
- moved U3 0.35 mm to (125.5, 114.2)
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Connections:
- net Net-(J1-D+) renamed /USB D+
- net Net-(J1-D-) renamed /USB D-
- J1 pad 1: Net-(J1-VBUS) -> /5V
- R5 pad 1: /5V -> /3V3
Routing:
- net /5V: track 0.00 -> 52.0 mm
- net /GND: track 0.00 -> 43.4 mm, vias 0 -> 14
- net /USB D+: track 0.00 -> 29.3 mm, vias 0 -> 2
- net /USB D-: track 0.00 -> 29.2 mm, vias 0 -> 2
- net /CS: track 0.00 -> 20.3 mm, vias 0 -> 1
- net /3V3: track 0.00 -> 17.6 mm, vias 0 -> 9
- net Net-(U3-DIO1): track 0.00 -> 13.1 mm, vias 0 -> 1
- net /CLK: track 0.00 -> 12.5 mm, vias 0 -> 1
- net /MOSI: track 0.00 -> 11.5 mm, vias 0 -> 1
- net /MISO: track 0.00 -> 10.8 mm, vias 0 -> 1
- net Net-(U3-DIO2): track 0.00 -> 7.05 mm, vias 0 -> 1
- net Net-(U2-XI): track 0.00 -> 6.62 mm
- net Net-(U2-XO): track 0.00 -> 4.38 mm
- net Net-(U2-V3): track 0.00 -> 2.81 mm
- net Net-(D1-A): track 0.00 -> 1.92 mm
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- added copper zone on In2.Cu, net /3V3
- added copper zone on In1.Cu, net /GND
Other:
- copper layers 2 -> 4
- board text added: "Akhil V :)"
- board text added: "JLCJLCJLCJLC"

Commit message: wip
Parts:
- removed TP1, TP2, TP3, TP4, TP5, TP6, TP7, TP8: TestPoint, TestPoint:TestPoint_Pad_1.0x1.0mm
- added J2: Conn_01x04_Female, Connector_PinSocket_2.54mm:PinSocket_1x04_P2.54mm_Vertical, F.Cu at (110.5, 120.6)
- R5: moved to F.Cu
- moved R2 14.6 mm to (110.6, 106.7)
- moved D1 14.4 mm to (112.0, 106.7)
- moved D4 14.4 mm to (114.0, 106.7)
- moved R3 14.1 mm to (115.6, 106.7)
- moved R5 1.89 mm to (127.8, 106.4), turned to 90 degrees
- moved C3 0.26 mm to (126.5, 106.4)
Routing:
- net /5V: track 52.0 -> 13.9 mm, vias 0 -> 3
- net /CS: track 20.3 -> 0.00 mm, vias 1 -> 0
- net /MOSI: track 11.5 -> 0.00 mm, vias 1 -> 0
- net /GND: track 43.4 -> 39.1 mm, vias 14 -> 12
- net /USB D-: track 29.2 -> 32.7 mm
- net /USB D+: track 29.3 -> 32.6 mm
- net /MISO: track 10.8 -> 7.67 mm
- net /CLK: track 12.5 -> 9.39 mm
- net /3V3: track 17.6 -> 18.2 mm, vias 9 -> 6
- net Net-(U3-nReset): track 1.66 -> 1.10 mm, vias 0 -> 1
- added copper zone on In2.Cu, net /5V
Other:
- board text removed: "3v3"
- board text removed: "5v"
- board text removed: "gnd"

Commit message: finished
Parts:
- moved R2 33.5 mm to (140.5, 121.9)
- moved D1 30.9 mm to (138.9, 121.9)
- moved D4 3.81 mm to (110.2, 106.7)
- moved R3 3.81 mm to (111.8, 106.7), turned to -90 degrees
- moved J2 0.43 mm to (110.1, 120.4)
- moved C2 0.30 mm to (108.8, 114.0)
Routing:
- net /CS: track 0.00 -> 38.6 mm, vias 0 -> 1
- net /MOSI: track 0.00 -> 28.7 mm, vias 0 -> 1
- net /MISO: track 7.67 -> 33.7 mm
- net /CLK: track 9.39 -> 18.3 mm
- net /3V3: track 18.2 -> 21.8 mm, vias 6 -> 7
- net /5V: track 13.9 -> 16.1 mm, vias 3 -> 5
- net Net-(U3-nReset): track 1.10 -> 2.80 mm
- net /GND: track 39.1 -> 39.9 mm, vias 12 -> 13
- net Net-(D4-K): track 1.63 -> 2.23 mm
Other:
- board text added: "Akhil V"
- board text added: "Steven G"
- board text removed: "Akhil V :)"

Commit message: merge main
Routing:
- net /MOSI: track 28.7 -> 27.4 mm
- net /CS: track 38.6 -> 38.0 mm
Changed lines of the file:
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@@
   (segment (start 123.698 116.84) (end 120.987 116.84) (width 0.3) (layer "F.Cu") (net 8))
   (segment (start 120.987 116.84) (end 120.86 116.967) (width 0.3) (layer "F.Cu") (net 8))
+  (segment (start 120.86 113.135) (end 120.86 116.967) (width 0.3) (layer "F.Cu") (net 8))
+  (segment (start 115.929 108.204) (end 120.86 113.135) (width 0.3) (layer "F.Cu") (net 8))
   (segment (start 111.7595 107.1915) (end 111.7595 107.6955) (width 0.3) (layer "F.Cu") (net 8))
-  (segment (start 112.268 108.204) (end 116.967 108.204) (width 0.3) (layer "F.Cu") (net 8))
-  (segment (start 120.86 112.097) (end 120.86 116.967) (width 0.3) (layer "F.Cu") (net 8))
+  (segment (start 120.86 116.967) (end 120.86 118.9) (width 0.3) (layer "F.Cu") (net 8))
+  (segment (start 112.268 108.204) (end 115.929 108.204) (width 0.3) (layer "F.Cu") (net 8))
   (segment (start 111.7595 107.6955) (end 112.268 108.204) (width 0.3) (layer "F.Cu") (net 8))
-  (segment (start 116.967 108.204) (end 120.86 112.097) (width 0.3) (layer "F.Cu") (net 8))
-  (segment (start 120.86 116.967) (end 120.86 118.9) (width 0.3) (layer "F.Cu") (net 8))
   (via (at 123.698 116.84) (size 0.8) (drill 0.4) (layers "F.Cu" "B.Cu") (net 8))
+  (segment (start 123.698 116.84) (end 124.6885 116.84) (width 0.3) (layer "B.Cu") (net 8))
+  (segment (start 123.698 116.84) (end 122.135 116.84) (width 0.3) (layer "B.Cu") (net 8))
+  (segment (start 124.6885 116.84) (end 128.4 120.5515) (width 0.3) (layer "B.Cu") (net 8))
+  (segment (start 116.533 118.925) (end 115.189 120.269) (width 0.3) (layer "B.Cu") (net 8))
   (segment (start 115.189 120.269) (end 115.189 120.396) (width 0.3) (layer "B.Cu") (net 8))
-  (segment (start 123.698 116.84) (end 124.6885 116.84) (width 0.3) (layer "B.Cu") (net 8))
-  (segment (start 124.6885 116.84) (end 128.4 120.5515) (width 0.3) (layer "B.Cu") (net 8))
-  (segment (start 116.332 119.126) (end 115.189 120.269) (width 0.3) (layer "B.Cu") (net 8))
-  (segment (start 123.698 116.84) (end 123.53925 116.84) (width 0.3) (layer "B.Cu") (net 8))
-  (segment (start 121.25325 119.126) (end 116.332 119.126) (width 0.3) (layer "B.Cu") (net 8))
-  (segment (start 123.53925 116.84) (end 121.25325 119.126) (width 0.3) (layer "B.Cu") (net 8))
+  (segment (start 120.05 118.925) (end 116.533 118.925) (width 0.3) (layer "B.Cu") (net 8))
   (segment (start 128.4 120.5515) (end 128.4 121.75) (width 0.3) (layer "B.Cu") (net 8))
+  (segment (start 122.135 116.84) (end 120.05 118.925) (width 0.3) (layer "B.Cu") (net 8))
   (segment (start 127.21 116.009) (end 127.21 118.9) (width 0.3) (layer "F.Cu") (net 9))
   (segment (start 127.1395 115.9385) (end 127.21 116.009) (width 0.3) (layer "F.Cu") (net 9))
   (via (at 127.1395 115.9385) (size 0.8) (drill 0.4) (layers "F.Cu" "B.Cu") (net 9))
+  (segment (start 114.768 118.15) (end 112.649 120.269) (width 0.3) (layer "B.Cu") (net 9))
+  (segment (start 121.249 115.951) (end 119.05 118.15) (width 0.3) (layer "B.Cu") (net 9))
   (segment (start 127.1395 115.9385) (end 127.127 115.951) (width 0.3) (layer "B.Cu") (net 9))
+  (segment (start 130.94 118.69) (end 130.94 121.75) (width 0.3) (layer "B.Cu") (net 9))
+  (segment (start 119.05 118.15) (end 114.768 118.15) (width 0.3) (layer "B.Cu") (net 9))
+  (segment (start 127.1395 115.9385) (end 128.1885 115.9385) (width 0.3) (layer "B.Cu") (net 9))
   (segment (start 112.649 120.269) (end 112.649 120.396) (width 0.3) (layer "B.Cu") (net 9))
-  (segment (start 130.94 116.5255) (end 130.94 121.75) (width 0.3) (layer "B.Cu") (net 9))
-  (segment (start 130.353 115.9385) (end 130.94 116.5255) (width 0.3) (layer "B.Cu") (net 9))
-  (segment (start 120.523 118.364) (end 114.554 118.364) (width 0.3) (layer "B.Cu") (net 9))
-  (segment (start 122.936 115.951) (end 120.523 118.364) (width 0.3) (layer "B.Cu") (net 9))
-  (segment (start 127.1395 115.9385) (end 130.353 115.9385) (width 0.3) (layer "B.Cu") (net 9))
-  (segment (start 127.127 115.951) (end 122.936 115.951) (width 0.3) (layer "B.Cu") (net 9))
-  (segment (start 114.554 118.364) (end 112.649 120.269) (width 0.3) (layer "B.Cu") (net 9))
+  (segment (start 127.127 115.951) (end 121.249 115.951) (width 0.3) (layer "B.Cu") (net 9))
+  (segment (start 128.1885 115.9385) (end 130.94 118.69) (width 0.3) (layer "B.Cu") (net 9))
   (segment (start 129.75 115.233) (end 129.75 118.9) (width 0.3) (layer "F.Cu") (net 10))
   (segment (start 129.794 115.189) (end 129.75 115.233) (width 0.3) (layer "F.Cu") (net 10))
   (via (at 129.794 115.189) (size 0.8) (drill 0.4) (layers "F.Cu" "B.Cu") (net 10))
-  (segment (start 132.21 116.716) (end 132.21 121.75) (width 0.3) (layer "B.Cu") (net 10))
-  (segment (start 119.888 117.602) (end 112.776 117.602) (width 0.3) (layer "B.Cu") (net 10))
-  (segment (start 112.776 117.602) (end 110.109 120.269) (width 0.3) (layer "B.Cu") (net 10))
-  (segment (start 129.794 115.189) (end 122.301 115.189) (width 0.3) (layer "B.Cu") (net 10))
-  (segment (start 130.683 115.189) (end 132.21 116.716) (width 0.3) (layer "B.Cu") (net 10))
-  (segment (start 122.301 115.189) (end 119.888 117.602) (width 0.3) (layer "B.Cu") (net 10))
-  (segment (start 129.794 115.189) (end 130.683 115.189) (width 0.3) (layer "B.Cu") (net 10))
-  (segment (start 110.109 120.269) (end 110.109 120.396) (width 0.3) (layer "B.Cu") (net 10))
+  (segment (start 130.339 115.189) (end 132.21 117.06) (width 0.3) (layer "B.Cu") (net 10))
+  (segment (start 118.3 117.325) (end 113.18 117.325) (width 0.3) (layer "B.Cu") (net 10))
+  (segment (start 132.21 117.06) (end 132.21 121.75) (width 0.3) (layer "B.Cu") (net 10))
+  (segment (start 129.794 115.189) (end 120.436 115.189) (width 0.3) (layer "B.Cu") (net 10))
+  (segment (start 129.794 115.189) (end 130.339 115.189) (width 0.3) (layer "B.Cu") (net 10))
+  (segment (start 120.436 115.189) (end 118.3 117.325) (width 0.3) (layer "B.Cu") (net 10))
+  (segment (start 113.18 117.325) (end 110.109 120.396) (width 0.3) (layer "B.Cu") (net 10))
   (segment (start 124.714 111.76) (end 124.714 111.252) (width 0.3) (layer "F.Cu") (net 16))
   (segment (start 125.878977 113.686977) (end 125.878977 112.924977) (width 0.3) (layer "F.Cu") (net 16))
