File: SX1280_USB_Adapter/SX1280_USB_Adapter.kicad_sch (KiCad schematic)
At the start: 16 parts, among them J1 USB_A, J2 Conn_01x07, J3 Conn_01x07, U1 AMS1117-3.3, U2 CH341a, U3 SX1280, Y1 12M

Commit message: schematic done
Parts:
- removed C1, C4: 20p, Capacitor_SMD:C_0603_1608Metric, symbol CH341Apro-rescue:C-Device
- removed C2, C5: 104, Capacitor_SMD:C_0603_1608Metric, symbol CH341Apro-rescue:C-Device
- removed C3: 472, Capacitor_SMD:C_0603_1608Metric, symbol CH341Apro-rescue:C-Device
- removed D1: Power, LED_SMD:LED_0603_1608Metric, symbol CH341Apro-rescue:LED_ALT-Device
- removed D2: RUN, LED_SMD:LED_0603_1608Metric, symbol CH341Apro-rescue:LED_ALT-Device
- removed J1: USB_A, connectors:USB_A_MALE_Generic, symbol CH341Apro-rescue:USB_A-Connector
- removed J2, J3: Conn_01x07, Connector_PinSocket_2.54mm:PinSocket_1x07_P2.54mm_Vertical, symbol CH341Apro-rescue:Conn_01x07-Connector_Generic
- removed R1: 0R, Resistor_SMD:R_0805_2012Metric, symbol CH341Apro-rescue:R-Device
- removed RN1: 222, Resistor_SMD:R_Array_Convex_4x0603, symbol CH341Apro-rescue:R_Pack04_Split-Device
- removed U1: AMS1117-3.3, Package_TO_SOT_SMD:SOT-223-3_TabPin2, symbol CH341Apro-rescue:AMS1117-3.3-Regulator_Linear
- removed Y1: 12M, Crystal:Crystal_HC49-U_Vertical, symbol CH341Apro-rescue:Crystal-Device
- added C1, C4: 20p, Capacitor_SMD:C_0402_1005Metric, symbol Device:C
- added C2, C5: 104, Capacitor_SMD:C_0402_1005Metric, symbol Device:C
- added C3: 47p2, Capacitor_SMD:C_0402_1005Metric, symbol Device:C
- added D1, D2, D3, D4: LED, LED_SMD:LED_0603_1608Metric, symbol Device:LED
- added J2: USB_A_PLUG, USB_PCB:USB_PCB, symbol armory-rescue:USB_A_PLUG
- added R1: 0, Resistor_SMD:R_0402_1005Metric, symbol Device:R
- added R2, R3, R4, R6: R330, Resistor_SMD:R_0402_1005Metric, symbol Device:R
- added R5: 1k, Resistor_SMD:R_0402_1005Metric, symbol Device:R
- added TP1, TP2, TP3, TP4, TP5, TP6, TP7: TestPoint, TestPoint:TestPoint_Pad_1.0x1.0mm, symbol Connector:TestPoint
- added U1: AMS1117-3.3, Package_TO_SOT_SMD:SOT-223-3_TabPin2, symbol Regulator_Linear:AMS1117-3.3
- added Y1: Crystal_GND24, Crystal:Crystal_SMD_3225-4Pin_3.2x2.5mm, symbol Device:Crystal_GND24
Connections:
- net Earth is gone; now on net GND: U2.12 (GND), U2.27 (~{TEN/BUSY/}WAIT), U3.2 (GND)
- net 3V3: now also C5.2, D4.2 (A), TP2.1, U1.2 (VO)
- net 5V: now also C2.2, R1.1, R2.1, R5.1, TP1.1, U1.3 (VI)
- net CLK: now also U3.5 (SCK), TP7.1
- net CS: now also U3.6 (NSS), R3.2, TP6.1
- net MISO: now also TP4.1
- net MOSI: now also TP5.1
- net at U2.9 (V3): now also C3.2
- net at U2.13 (XI): now also C1.2, Y1.1
- net at U2.11 (UD-): now also J2.2 (D-)
- net at U2.10 (UD+): now also J2.3 (D+)
- net at U2.14 (XO): now also C4.2, Y1.3
- net at U3.11 (DIO1): now also R4.1
- net at U3.12 (DIO2): now also R6.1
- net GND: now reaches U3.14 (GND)
- net GND: now also U3.7 (GND), U3.8 (GND), C1.1, C2.1, C3.1, C4.1, C5.1, D1.1 (K), D2.1 (K), D3.1 (K), J2.4 (GND), TP3.1, U1.1 (GND), Y1.2, Y1.4
- net at U3.9 (nReset): now also R5.2
- net RXD: no longer names the net of U2.6 (RXD/PEMP/USERDEF)
- net SDA: no longer names the net of U2.23 (SDA)
- net TXD: no longer names the net of U2.5 (TXD/~{ERR/USERDEF})
- new net: J2.1 (VBUS), R1.2
- new net: D2.2 (A), R4.2
- new net: D3.2 (A), R6.2
- new net: D1.2 (A), R2.2
- new net: D4.1 (K), R3.1
- no-connect marks 12 -> 18
Other:
- moved on the sheet: U2, U3

Commit message: update layout
Parts:
- added TP8: TestPoint, TestPoint:TestPoint_Pad_1.0x1.0mm, symbol Connector:TestPoint
Connections:
- net GND: now also TP8.1
Changed lines of the file:
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@@
   (junction (at 195.58 111.76) (diameter 0) (color 0 0 0 0)
+  )
+  (junction (at 217.678 104.14) (diameter 0) (color 0 0 0 0)
   )
   (junction (at 114.3 81.28) (diameter 0) (color 0 0 0 0)
@@
     (stroke (width 0) (type default))
   )
+  (wire (pts (xy 217.678 104.14) (xy 226.06 104.14))
+    (stroke (width 0) (type default))
+  )
   (wire (pts (xy 163.83 109.22) (xy 175.26 109.22))
     (stroke (width 0) (type default))
@@
     (stroke (width 0) (type default))
   )
+  (wire (pts (xy 217.678 117.094) (xy 226.187 117.094))
+    (stroke (width 0) (type default))
+  )
   (wire (pts (xy 212.09 140.97) (xy 212.09 151.13))
     (stroke (width 0) (type default))
@@
     (stroke (width 0) (type default))
   )
+  (wire (pts (xy 217.678 104.14) (xy 217.678 117.094))
+    (stroke (width 0) (type default))
+  )
   (wire (pts (xy 222.25 140.97) (xy 222.25 142.24))
     (stroke (width 0) (type default))
@@
     (stroke (width 0) (type default))
   )
-  (wire (pts (xy 212.09 104.14) (xy 226.06 104.14))
+  (wire (pts (xy 212.09 104.14) (xy 217.678 104.14))
     (stroke (width 0) (type default))
   )
@@
         )
       )
+    )
+  )
+  (symbol (lib_id "Connector:TestPoint") (at 226.187 117.094 270) (unit 1)
+    (in_bom yes) (on_board yes) (dnp no)
+    (property "Reference" "TP8" (at 231.267 116.459 90)
+      (effects (font (size 1.27 1.27)) (justify left))
+    )
+    (property "Value" "TestPoint" (at 236.982 117.094 90)
+      (effects (font (size 1.27 1.27)) (justify left))
+    )
+    (property "Footprint" "TestPoint:TestPoint_Pad_1.0x1.0mm" (at 226.187 122.174 0)
+      (effects (font (size 1.27 1.27)) hide)
+    )
+    (property "Datasheet" "~" (at 226.187 122.174 0)
+      (effects (font (size 1.27 1.27)) hide)
+    )
+    (pin "1")
+    (instances
+      (project "SX1280_USB_Adapter"
+        (path "/a4f28170-029d-4dad-baf4-7640b7dbeb52"
+          (reference "TP8") (unit 1)
+        )
+      )

Commit message: layout finished
Parts:
- removed R1: 0, Resistor_SMD:R_0402_1005Metric, symbol Device:R
Connections:
- net 3V3: now also R5.1
- net 5V: now also J2.1 (VBUS); no longer R5.1
- net USB D-: now reaches J2.2 (D-), U2.11 (UD-)
- net USB D+: now reaches J2.3 (D+), U2.10 (UD+)
Changed lines of the file:
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@@
   (junction (at 109.22 151.13) (diameter 0) (color 0 0 0 0)
   )
+  (junction (at 214.63 101.6) (diameter 0) (color 0 0 0 0)
+  )
   (junction (at 171.45 140.97) (diameter 0) (color 0 0 0 0)
   )
@@
   )
   (junction (at 212.09 151.13) (diameter 0) (color 0 0 0 0)
-  )
-  (junction (at 214.63 99.06) (diameter 0) (color 0 0 0 0)
   )
   (junction (at 105.41 151.13) (diameter 0) (color 0 0 0 0)
@@
     (stroke (width 0) (type default))
   )
-  (wire (pts (xy 214.63 99.06) (xy 226.06 99.06))
+  (wire (pts (xy 205.74 99.06) (xy 226.06 99.06))
     (stroke (width 0) (type default))
   )
@@
     (stroke (width 0) (type default))
   )
-  (wire (pts (xy 205.74 99.06) (xy 214.63 99.06))
-    (stroke (width 0) (type default))
-  )
   (wire (pts (xy 163.83 121.92) (xy 170.18 121.92))
     (stroke (width 0) (type default))
@@
     (stroke (width 0) (type default))
   )
+  (wire (pts (xy 214.63 101.6) (xy 214.63 119.38))
+    (stroke (width 0) (type default))
+  )
   (wire (pts (xy 80.01 151.13) (xy 86.36 151.13))
     (stroke (width 0) (type default))
@@
     (stroke (width 0) (type default))
   )
-  (wire (pts (xy 214.63 99.06) (xy 214.63 119.38))
-    (stroke (width 0) (type default))
-  )
   (wire (pts (xy 212.09 104.14) (xy 217.678 104.14))
     (stroke (width 0) (type default))
@@
     (stroke (width 0) (type default))
   )
-  (wire (pts (xy 77.47 74.93) (xy 77.47 57.15))
+  (wire (pts (xy 77.47 57.15) (xy 77.47 118.11))
     (stroke (width 0) (type default))
   )
@@
     (stroke (width 0) (type default))
   )
+  (wire (pts (xy 114.3 69.85) (xy 114.3 67.31))
+    (stroke (width 0) (type default))
+  )
+  (wire (pts (xy 212.09 151.13) (xy 222.25 151.13))
+    (stroke (width 0) (type default))
+  )
+  (wire (pts (xy 86.36 57.15) (xy 114.3 57.15))
+    (stroke (width 0) (type default))
+  )
+  (wire (pts (xy 207.01 138.43) (xy 214.63 138.43))
+    (stroke (width 0) (type default))
+  )
+  (wire (pts (xy 86.36 72.39) (xy 86.36 74.93))
+    (stroke (width 0) (type default))
+  )
+  (wire (pts (xy 114.3 77.47) (xy 114.3 81.28))
+    (stroke (width 0) (type default))
+  )
+  (wire (pts (xy 214.63 127) (xy 214.63 138.43))
+    (stroke (width 0) (type default))
+  )
+  (wire (pts (xy 205.74 57.15) (xy 205.74 99.06))
+    (stroke (width 0) (type default))
+  )
+  (wire (pts (xy 195.58 76.2) (xy 195.58 90.17))
+    (stroke (width 0) (type default))
+  )
+  (wire (pts (xy 207.01 125.73) (xy 212.09 125.73))
+    (stroke (width 0) (type default))
+  )
+  (wire (pts (xy 109.22 135.89) (xy 109.22 130.81))
+    (stroke (width 0) (type default))
+  )
+  (wire (pts (xy 119.38 151.13) (xy 114.3 151.13))
+    (stroke (width 0) (type default))
+  )
+  (wire (pts (xy 214.63 101.6) (xy 226.06 101.6))
+    (stroke (width 0) (type default))
+  )
+  (wire (pts (xy 74.93 106.68) (xy 80.01 106.68))
+    (stroke (width 0) (type default))
+  )
+  (wire (pts (xy 119.38 121.92) (xy 121.92 121.92))
+    (stroke (width 0) (type default))
+  )
+  (wire (pts (xy 212.09 104.14) (xy 212.09 125.73))
+    (stroke (width 0) (type default))
+  )
+  (wire (pts (xy 163.83 88.9) (xy 172.72 88.9))
+    (stroke (width 0) (type default))
+  )
+  (wire (pts (xy 139.7 67.31) (xy 177.8 67.31))
+    (stroke (width 0) (type default))
+  )
   (wire (pts (xy 74.93 114.3) (xy 121.92 114.3))
     (stroke (width 0) (type default))
   )
-  (wire (pts (xy 114.3 69.85) (xy 114.3 67.31))
-    (stroke (width 0) (type default))
-  )
-  (wire (pts (xy 212.09 151.13) (xy 222.25 151.13))
-    (stroke (width 0) (type default))
-  )
-  (wire (pts (xy 86.36 57.15) (xy 114.3 57.15))
-    (stroke (width 0) (type default))
-  )
-  (wire (pts (xy 207.01 138.43) (xy 214.63 138.43))
-    (stroke (width 0) (type default))
-  )
-  (wire (pts (xy 86.36 72.39) (xy 86.36 74.93))
-    (stroke (width 0) (type default))
-  )
-  (wire (pts (xy 77.47 82.55) (xy 77.47 118.11))
-    (stroke (width 0) (type default))
-  )
-  (wire (pts (xy 114.3 77.47) (xy 114.3 81.28))
-    (stroke (width 0) (type default))
-  )
-  (wire (pts (xy 214.63 127) (xy 214.63 138.43))
-    (stroke (width 0) (type default))
-  )
-  (wire (pts (xy 205.74 57.15) (xy 205.74 99.06))
-    (stroke (width 0) (type default))
-  )
-  (wire (pts (xy 195.58 76.2) (xy 195.58 90.17))
-    (stroke (width 0) (type default))
-  )
-  (wire (pts (xy 207.01 125.73) (xy 212.09 125.73))
-    (stroke (width 0) (type default))
-  )
-  (wire (pts (xy 109.22 135.89) (xy 109.22 130.81))
-    (stroke (width 0) (type default))
-  )
-  (wire (pts (xy 119.38 151.13) (xy 114.3 151.13))
-    (stroke (width 0) (type default))
-  )
-  (wire (pts (xy 74.93 106.68) (xy 80.01 106.68))
-    (stroke (width 0) (type default))
-  )
-  (wire (pts (xy 119.38 121.92) (xy 121.92 121.92))
-    (stroke (width 0) (type default))
-  )
-  (wire (pts (xy 212.09 104.14) (xy 212.09 125.73))
-    (stroke (width 0) (type default))
-  )
-  (wire (pts (xy 163.83 88.9) (xy 172.72 88.9))
-    (stroke (width 0) (type default))
-  )
-  (wire (pts (xy 139.7 67.31) (xy 177.8 67.31))
-    (stroke (width 0) (type default))
-  )
   (wire (pts (xy 171.45 91.44) (xy 171.45 128.27))
     (stroke (width 0) (type default))
   )
-  (wire (pts (xy 203.2 101.6) (xy 226.06 101.6))
+  (wire (pts (xy 203.2 101.6) (xy 214.63 101.6))
     (stroke (width 0) (type default))
   )
@@
     (effects (font (size 1.27 1.27)) (justify left bottom))
   )
+  (label "USB D-" (at 82.55 114.3 0) (fields_autoplaced)
+    (effects (font (size 1.27 1.27)) (justify left bottom))
+  )
   (label "MOSI" (at 165.1 109.22 0) (fields_autoplaced)
     (effects (font (size 1.27 1.27)) (justify left bottom))
@@
   )
   (label "MISO" (at 165.1 104.14 0) (fields_autoplaced)
+    (effects (font (size 1.27 1.27)) (justify left bottom))
+  )
+  (label "USB D+" (at 82.55 110.49 0) (fields_autoplaced)
     (effects (font (size 1.27 1.27)) (justify left bottom))
   )
@@
         )
       )
-    )
-  )
-  (symbol (lib_id "Device:R") (at 77.47 78.74 0) (unit 1)
-    (in_bom yes) (on_board yes) (dnp no) (fields_autoplaced)
-    (property "Reference" "R1" (at 80.01 78.105 0)
-      (effects (font (size 1.27 1.27)) (justify left))
-    )
-    (property "Value" "0" (at 80.01 80.645 0)
-      (effects (font (size 1.27 1.27)) (justify left))
-    )
-    (property "Footprint" "Resistor_SMD:R_0402_1005Metric" (at 75.692 78.74 90)
-      (effects (font (size 1.27 1.27)) hide)
-    )
-    (property "Datasheet" "~" (at 77.47 78.74 0)
-      (effects (font (size 1.27 1.27)) hide)
-    )
-    (pin "1")
-    (pin "2")
-    (instances
-      (project "SX1280_USB_Adapter"
-        (path "/a4f28170-029d-4dad-baf4-7640b7dbeb52"
-          (reference "R1") (unit 1)
-        )
-      )

Commit message: wip
Parts:
- removed TP1, TP2, TP3, TP4, TP5, TP6, TP7, TP8: TestPoint, TestPoint:TestPoint_Pad_1.0x1.0mm, symbol Connector:TestPoint
- added J2: Conn_01x04_Female, Connector_PinSocket_2.54mm:PinSocket_1x04_P2.54mm_Vertical, symbol Connector:Conn_01x04_Female
Connections:
- net CLK: now also J2.4 (Pin_4)
- net CS: now also J2.3 (Pin_3)
- net MISO: now also J2.1 (Pin_1)
- net MOSI: now also J2.2 (Pin_2)
- net 3V3: no longer names the net of C5.2, D4.2 (A), R5.1, U1.2 (VO), U3.1 (VCC)
- net 5V: no longer names the net of C2.2, J2.1 (VBUS), R2.1, U1.3 (VI), U2.28 (VCC)
- net GND: no longer names the net of C1.1, C2.1, C3.1, C4.1, C5.1, D1.1 (K), D2.1 (K), D3.1 (K), J2.4 (GND), U1.1 (GND), U2.12 (GND), U2.27 (~{TEN/BUSY/}WAIT), U3.14 (GND), U3.2 (GND), U3.7 (GND), U3.8 (GND), Y1.2, Y1.4

Commit message: build output files
Parts:
- C1, C4: value 20p -> 18p; LCSC (none) -> C1549
- C2, C5: LCSC (none) -> C19702
- C3: LCSC (none) -> C15195
- D1, D2, D3, D4: LCSC (none) -> C72041
- R2, R3, R4, R6: LCSC (none) -> C25104
- R5: value 1k -> 330; LCSC (none) -> C25104
- U1: LCSC (none) -> C6186
- U2: LCSC (none) -> C13517
Changed lines of the file:
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@@
+      (effects (font (size 1.27 1.27)) hide)
+    )
+    (property "LCSC" "C25104" (at 222.25 137.16 0)
       (effects (font (size 1.27 1.27)) hide)
     )
@@
       (effects (font (size 1.27 1.27)) hide)
     )
+    (property "LCSC" "C72041" (at 237.49 146.05 90)
+      (effects (font (size 1.27 1.27)) hide)
+    )
     (pin "1")
     (pin "2")
@@
       (effects (font (size 1.27 1.27)) hide)
     )
+    (property "LCSC" "C25104" (at 237.49 138.43 0)
+      (effects (font (size 1.27 1.27)) hide)
+    )
     (pin "1")
     (pin "2")
@@
       (effects (font (size 1.27 1.27)) hide)
     )
+    (property "LCSC" "C72041" (at 86.36 78.74 90)
+      (effects (font (size 1.27 1.27)) hide)
+    )
     (pin "1")
     (pin "2")
@@
       (effects (font (size 1.27 1.27)) (justify right))
     )
-    (property "Value" "20p" (at 123.19 141.605 0)
+    (property "Value" "18p" (at 123.19 141.605 0)
       (effects (font (size 1.27 1.27)) (justify right))
     )
@@
     )
     (property "Datasheet" "~" (at 119.38 139.7 0)
+      (effects (font (size 1.27 1.27)) hide)
+    )
+    (property "LCSC" "C1549" (at 119.38 139.7 0)
       (effects (font (size 1.27 1.27)) hide)
     )
@@
       (effects (font (size 1.27 1.27)) hide)
     )
+    (property "LCSC" "C72041" (at 195.58 72.39 90)
+      (effects (font (size 1.27 1.27)) hide)
+    )
     (pin "1")
     (pin "2")
@@
       (effects (font (size 1.27 1.27)) hide)
     )
+    (property "LCSC" "C19702" (at 114.3 73.66 0)
+      (effects (font (size 1.27 1.27)) hide)
+    )
     (pin "1")
     (pin "2")
@@
       (effects (font (size 1.27 1.27)) hide)
     )
+    (property "LCSC" "C6186" (at 127 67.31 0)
+      (effects (font (size 1.27 1.27)) hide)
+    )
     (pin "1")
     (pin "2")
@@
     )
     (property "Datasheet" "~" (at 195.58 93.98 0)
+      (effects (font (size 1.27 1.27)) hide)
+    )
+    (property "LCSC" "C25104" (at 195.58 93.98 0)
       (effects (font (size 1.27 1.27)) hide)
     )
@@
       (effects (font (size 1.27 1.27)) hide)
     )
+    (property "LCSC" "C25104" (at 86.36 68.58 0)
+      (effects (font (size 1.27 1.27)) hide)
+    )
     (pin "1")
     (pin "2")
@@
       (effects (font (size 1.27 1.27)) hide)
     )
+    (property "LCSC" "C15195" (at 114.3 109.22 90)
+      (effects (font (size 1.27 1.27)) hide)
+    )
     (pin "1")
     (pin "2")
@@
       (effects (font (size 1.27 1.27)) hide)
     )
+    (property "LCSC" "C72041" (at 222.25 146.05 90)
+      (effects (font (size 1.27 1.27)) hide)
+    )
     (pin "1")
     (pin "2")
@@
       (effects (font (size 1.27 1.27)) hide)
     )
+    (property "LCSC" "C19702" (at 139.7 73.66 0)
+      (effects (font (size 1.27 1.27)) hide)
+    )
     (pin "1")
     (pin "2")
@@
       (effects (font (size 1.27 1.27)) (justify left))
     )
-    (property "Value" "1k" (at 217.17 125.095 0)
+    (property "Value" "330" (at 217.17 125.095 0)
       (effects (font (size 1.27 1.27)) (justify left))
     )
@@
     )
     (property "Datasheet" "~" (at 214.63 123.19 0)
+      (effects (font (size 1.27 1.27)) hide)
+    )
+    (property "LCSC" "C25104" (at 214.63 123.19 0)
       (effects (font (size 1.27 1.27)) hide)
     )
@@
     )
     (property "Datasheet" "" (at 132.08 101.6 0)
+      (effects (font (size 1.27 1.27)) hide)
+    )
+    (property "LCSC" "C13517" (at 142.24 105.41 0)
       (effects (font (size 1.27 1.27)) hide)
     )
@@
       (effects (font (size 1.27 1.27)) (justify right))
     )
-    (property "Value" "20p" (at 113.03 141.605 0)
+    (property "Value" "18p" (at 113.03 141.605 0)
       (effects (font (size 1.27 1.27)) (justify right))
     )
@@
       (effects (font (size 1.27 1.27)) hide)
     )
+    (property "LCSC" "C1549" (at 109.22 139.7 0)
+      (effects (font (size 1.27 1.27)) hide)
+    )
