File: PowerBoard/Flyback_HV.kicad_sch (KiCad schematic)
At the start: 63 parts, among them Q2 IRFR3410TRPBF, Q3 FGH50T65SQD-F155, Q5 TN2130K1-G, Q6 IPD60R3K4CEAUMA1, Q7 FGH50T65SQD-F155, T1 DA2034, U2 LT3750, U4 MCP14A0454-E/SN

Commit message: chicker v1.0 ordered
Parts:
- removed TP21: VGATE, bots:TestPoint_Pad_1.0x1.0mm, symbol bots:TestPoint_1x1
- added R49: R_0OHM_JUMPER, bots:R_0603_1608Metric, symbol bots:R_0OHM_JUMPER
Connections:
- net V_GATE_Q2: no longer Q2.1 (G), U2.7 (GATE)
- new net: R49.1, U2.7 (GATE)
- new net: Q2.1 (G), R49.2
Other:
- moved on the sheet: Q2
Changed lines of the file:
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@@
   (junction (at 54.61 39.37) (diameter 0) (color 0 0 0 0)
   )
-  (junction (at 95.25 59.69) (diameter 0) (color 0 0 0 0)
-  )
   (junction (at 74.93 123.19) (diameter 0) (color 0 0 0 0)
   )
@@
     (stroke (width 0) (type default))
   )
-  (wire (pts (xy 95.25 59.69) (xy 96.52 59.69))
-    (stroke (width 0) (type default))
-  )
   (wire (pts (xy 60.96 53.34) (xy 60.96 58.42))
     (stroke (width 0) (type default))
@@
     (stroke (width 0) (type default))
   )
+  (wire (pts (xy 99.06 59.69) (xy 100.33 59.69))
+    (stroke (width 0) (type default))
+  )
   (wire (pts (xy 49.53 110.49) (xy 49.53 114.3))
     (stroke (width 0) (type default))
@@
     (stroke (width 0) (type default))
   )
+  (wire (pts (xy 107.95 67.31) (xy 104.14 67.31))
+    (stroke (width 0) (type default))
+  )
   (wire (pts (xy 60.96 74.93) (xy 60.96 76.2))
     (stroke (width 0) (type default))
@@
     (stroke (width 0) (type default))
   )
-  (wire (pts (xy 104.14 67.31) (xy 104.14 64.77))
+  (wire (pts (xy 107.95 67.31) (xy 107.95 64.77))
     (stroke (width 0) (type default))
   )
@@
     (stroke (width 0) (type default))
   )
+  (wire (pts (xy 107.95 54.61) (xy 104.14 54.61))
+    (stroke (width 0) (type default))
+  )
   (wire (pts (xy 90.17 31.75) (xy 118.11 31.75))
     (stroke (width 0) (type default))
@@
     (stroke (width 0) (type default))
   )
-  (wire (pts (xy 91.44 59.69) (xy 95.25 59.69))
-    (stroke (width 0) (type default))
-  )
   (wire (pts (xy 133.35 44.45) (xy 133.35 46.99))
     (stroke (width 0) (type default))
@@
     (effects (font (size 1.27 1.27)) (justify left bottom))
   )
-  (label "V_GATE_Q2" (at 92.71 59.69 0) (fields_autoplaced)
+  (label "V_GATE_Q2" (at 97.79 59.69 0) (fields_autoplaced)
     (effects (font (size 1.27 1.27)) (justify left bottom))
   )
@@
     (effects (font (size 1.27 1.27)) (justify left bottom))
   )
-  (label "VSOURCE" (at 104.14 67.31 0) (fields_autoplaced)
+  (label "VSOURCE" (at 107.95 67.31 0) (fields_autoplaced)
     (effects (font (size 1.27 1.27)) (justify left bottom))
   )
@@
     )
   )
-  (symbol (lib_id "bots:TestPoint_1x1") (at 95.25 59.69 180) (unit 1)
-    (in_bom no) (on_board yes) (dnp no)
-    (property "Reference" "TP21" (at 95.25 64.77 0)
-      (effects (font (size 1.27 1.27)) (justify left))
-    )
-    (property "Value" "VGATE" (at 93.98 62.23 0)
-      (effects (font (size 1.27 1.27)) (justify left))
-    )
-    (property "Footprint" "bots:TestPoint_Pad_1.0x1.0mm" (at 90.17 59.69 0)
-      (effects (font (size 1.27 1.27)) hide)
-    )
-    (property "Datasheet" "~" (at 90.17 59.69 0)
-      (effects (font (size 1.27 1.27)) hide)
-    )
-    (pin "1")
-    (instances
-      (project "POWER_BOARD"
-        (path "/1a9ce3e8-a091-496c-9c5f-e7b2eb60e275/aa68550e-c35d-4fef-b4e5-f1eb6225215f"
-          (reference "TP21") (unit 1)
-        )
-        (path "/1a9ce3e8-a091-496c-9c5f-e7b2eb60e275/13b16574-f046-4bb6-b573-f06681d59f31"
-          (reference "TP18") (unit 1)
-        )
-      )
-    )
-  )
   (symbol (lib_id "power:GNDPWR") (at 31.75 114.3 0) (unit 1)
     (in_bom yes) (on_board yes) (dnp no) (fields_autoplaced)
@@
     )
   )
+  (symbol (lib_id "bots:R_0OHM_JUMPER") (at 95.25 59.69 90) (unit 1)
+    (in_bom yes) (on_board yes) (dnp no)
+    (property "Reference" "R49" (at 93.98 57.15 90)
+      (effects (font (size 1.27 1.27)))
+    )
+    (property "Value" "R_0OHM_JUMPER" (at 95.25 59.69 90)
+      (effects (font (size 1.27 1.27)))
+    )
+    (property "Footprint" "bots:R_0603_1608Metric" (at 95.25 61.468 90)
+      (effects (font (size 1.27 1.27)) hide)
+    )
+    (property "Datasheet" "~" (at 95.25 59.69 0)
+      (effects (font (size 1.27 1.27)) hide)
+    )
+    (property "MPN" "0603WAF0000T5E" (at 95.25 59.69 0)
+      (effects (font (size 1.27 1.27)) hide)
+    )
+    (property "Manufacturer" "UNI-ROYAL(Uniroyal Elec)" (at 95.25 59.69 0)
+      (effects (font (size 1.27 1.27)) hide)
+    )
+    (property "Price" "0.001" (at 95.25 59.69 0)
+      (effects (font (size 1.27 1.27)) hide)
+    )
+    (property "JLC" "0603" (at 95.25 59.69 0)
+      (effects (font (size 1.27 1.27)) hide)
+    )
+    (property "LCSC" "C21189" (at 95.25 59.69 0)
+      (effects (font (size 1.27 1.27)) hide)
+    )
+    (property "JLC Extended" "no" (at 95.25 59.69 0)
+      (effects (font (size 1.27 1.27)) hide)
+    )
+    (pin "1")
+    (pin "2")
+    (instances
+      (project "POWER_BOARD"
+        (path "/1a9ce3e8-a091-496c-9c5f-e7b2eb60e275/aa68550e-c35d-4fef-b4e5-f1eb6225215f"
+          (reference "R49") (unit 1)
+        )
+      )
+    )
+  )
   (symbol (lib_id "bots:C_0.1u") (at 25.4 110.49 0) (unit 1)
     (in_bom yes) (on_board yes) (dnp no) (fields_autoplaced)
@@
     )
   )
-  (symbol (lib_id "bots:IRFR3410TRPBF") (at 101.6 59.69 0) (unit 1)
+  (symbol (lib_id "bots:IRFR3410TRPBF") (at 105.41 59.69 0) (unit 1)
     (in_bom yes) (on_board yes) (dnp no) (fields_autoplaced)
-    (property "Reference" "Q2" (at 107.95 58.42 0)
+    (property "Reference" "Q2" (at 111.76 58.42 0)
       (effects (font (size 1.27 1.27)) (justify left))
     )
-    (property "Value" "IRFR3410TRPBF" (at 107.95 60.96 0)
+    (property "Value" "IRFR3410TRPBF" (at 111.76 60.96 0)
       (effects (font (size 1.27 1.27)) (justify left))
     )
-    (property "Footprint" "bots:DPAK-3_ONS" (at 106.68 61.595 0)
+    (property "Footprint" "bots:DPAK-3_ONS" (at 110.49 61.595 0)
       (effects (font (size 1.27 1.27) italic) (justify left) hide)
     )
-    (property "Datasheet" "https://www.st.com/resource/en/datasheet/stb15n80k5.pdf" (at 101.6 59.69 0)
+    (property "Datasheet" "https://www.st.com/resource/en/datasheet/stb15n80k5.pdf" (at 105.41 59.69 0)
       (effects (font (size 1.27 1.27)) (justify left) hide)
     )
-    (property "MPN" "IRFR3410TRPBF" (at 101.6 59.69 0)
+    (property "MPN" "IRFR3410TRPBF" (at 105.41 59.69 0)
       (effects (font (size 1.27 1.27)) hide)
     )
-    (property "Manufacturer" "onsemi" (at 101.6 59.69 0)
+    (property "Manufacturer" "onsemi" (at 105.41 59.69 0)
       (effects (font (size 1.27 1.27)) hide)
     )
-    (property "Price" "0.465" (at 101.6 59.69 0)
+    (property "Price" "0.465" (at 105.41 59.69 0)
       (effects (font (size 1.27 1.27)) hide)
     )
-    (property "JLC" "TO-252" (at 101.6 59.69 0)
+    (property "JLC" "TO-252" (at 105.41 59.69 0)
       (effects (font (size 1.27 1.27)) hide)
     )
-    (property "LCSC" "C3016" (at 101.6 59.69 0)
+    (property "LCSC" "C3016" (at 105.41 59.69 0)
       (effects (font (size 1.27 1.27)) hide)
     )
-    (property "Description" "N-Channel 150 V 50A (Tc) 160W (Tj) Surface Mount TO-252AA" (at 101.6 59.69 0)
+    (property "Description" "N-Channel 150 V 50A (Tc) 160W (Tj) Surface Mount TO-252AA" (at 105.41 59.69 0)
       (effects (font (size 1.27 1.27)) hide)
     )
-    (property "JLC Extended" "yes" (at 101.6 59.69 0)
+    (property "JLC Extended" "yes" (at 105.41 59.69 0)
       (effects (font (size 1.27 1.27)) hide)
     )

Commit message: update
Parts:
- R48: now not fitted; now left out of the parts list
Changed lines of the file:
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@@
   )
   (symbol (lib_id "bots:2k_35W") (at 275.59 104.14 0) (unit 1)
-    (in_bom yes) (on_board yes) (dnp no) (fields_autoplaced)
+    (in_bom no) (on_board yes) (dnp yes) (fields_autoplaced)
     (property "Reference" "R48" (at 273.05 102.87 0)
       (effects (font (size 1.27 1.27)) (justify right))
