File: FacePlate/FacePlate.kicad_sch (KiCad schematic)
At the start: 38 parts, among them J1 Conn_01x02_Pin, J10 JST_XH_A_1x4, J11 Conn_01x02_Pin, J2 Conn_02x20_Odd_Even, J3 JST_XH_A_1x4, J4 Conn_01x02_Pin, J5 JST_BM08B-GHS-TBT, J6 JST_BM08B-GHS-TBT, J7 JST_XH_A_1x4, J8 JST_XH_A_1x4, J9 JST_XH_A_1x4, U1 GC9A, U2 GC9A, U7 AMS1117-3.3

Commit message: fix models
Parts:
- J10, J7, J8, J9: value JST_XH_A_1x4 -> STEMMA_QT; footprint bots:JST_XH_B4B-XH-AM_1x04_P2.50mm_Vertical -> Connector_JST:JST_SH_BM04B-SRSS-TB_1x04-1MP_P1.00mm_Vertical
- J4: renamed from J3; value JST_XH_A_1x4 -> JST_GH_BM04B-GHS-TBT_1x04; footprint bots:JST_XH_B4B-XH-AM_1x04_P2.50mm_Vertical -> Connector_JST:JST_GH_BM04B-GHS-TBT_1x04-1MP_P1.25mm_Vertical
- renumbered C2 to C1, C4 to C2, C1 to C3, C3 to C4, C16 to C5, C17 to C6, H4 to H1, H6 to H2, H1 to H3, H5 to H4, H2 to H5, H7 to H6, H3 to H7, J11 to J1, J6 to J11, J1 to J3, J4 to J5, J5 to J6, R19 to R1, R21 to R10, R22 to R2, R23 to R3, R24 to R4, R26 to R5, R28 to R6, R25 to R7, R27 to R8, R20 to R9, U7 to U3

Commit message: old-annotated schematic
Parts:
- removed C6: C, symbol Device:C
- added C17: 22u, bots:C_0603_1608Metric, symbol bots:C_22u
- renumbered C3 to C1, C5 to C16, C1 to C2, C4 to C3, C2 to C4, J8 to J, J11 to J, J6 to J, J10 to J, J1 to J, J7 to J, J9 to J, J3 to J1, J4 to J3, J5 to J4, R1 to R19, R9 to R20, R10 to R21, R2 to R22, R3 to R23, R4 to R24, R7 to R25, R5 to R26, R8 to R27, R6 to R28, U3 to U7
Connections:
- net +3.3V: now also C17.1
- net GND: now also C17.2
