File: Chicker/RP2040_CAN_FLASH.kicad_sch (KiCad schematic)
At the start: 59 parts, among them J1 JST_B3B-XH-A, J2 USB4145-03-0170-C_REVA2, J3 JST_BM04B-GHS-TBT, J4 JST_2P_LIMITSW, J5 Conn_02x10_Counter_Clockwise, U1 RPI2040, U10 PTS647SM38SMTR2LFS, U5 W25Q16JVSNIQ, U6 SN65HVD233, U7 MCP2515-xST, U9 PTS647SM38SMTR2LFS, Y1 ABM3-12.000MHZ-D2Y-T, Y2 ABM3-8.000MHZ-D2Y-T

Commit message: update for v1.1
Parts:
- removed C?: 0.1u, bots:C_0603_1608Metric, symbol bots:C_0.1u
- removed R20, R21: 33R, bots:R_0603_1608Metric, symbol bots:R_33R
- added C?: 1u, bots:C_0603_1608Metric, symbol bots:C_1u
- added R13: 200R, bots:R_0603_1608Metric, symbol thebots_symlib:R_200R
- added R14: R_27.4R, bots:R_0603_1608Metric, symbol thebots_symlib:R_27.4R
- added R20, R21: 27R, bots:R_0603_1608Metric, symbol thebots_symlib:R_27R
- added R? (x2): 5.1k, bots:R_0603_1608Metric, symbol bots:R_5.1k
Connections:
- net +3.3V: now also R13.2, R?.2; no longer U1.43 (ADC_AVDD)
- net D+: now also R20.2
- net D-: now also R21.2
- net DR+: now also R20.1
- net DR-: now also R21.1
- net GND: now also C?.2
- net GPIO28_ADC2 renamed 3v3_ref
- net 3v3_ref: now also R?.1
- new net AGND_ref: C?.1, R13.1, U1.43 (ADC_AVDD)
Other:
- moved on the sheet: C?

Commit message: chicker updates
Parts:
- removed R14: R_27.4R, bots:R_0603_1608Metric, symbol thebots_symlib:R_27.4R
- removed R? (x2): 5.1k, bots:R_0603_1608Metric, symbol bots:R_5.1k
- added R1: 100k, bots:R_0603_1608Metric, symbol bots:R_100k
Connections:
- net +3.3V: now also R1.2
- net 3v3_ref: now also R1.1
- net GPIO27_ADC1: no longer U1.39 (GPIO27/ADC1)
- net GPIO29_ADC3: no longer U1.41 (GPIO29/ADC3)
- new net 5V_LEVEL: U1.39 (GPIO27/ADC1)
- new net HV_SENSE: U1.41 (GPIO29/ADC3)
Other:
- moved on the sheet: TP1, U10, U9
