File: pmw3360-pcb-main/pmw3360_pcb_jst/pmw3360_pcb_jst.kicad_sch (KiCad schematic)
At the start: 20 parts, among them J1 Conn_01x08, U1 PMW3360DM-T2QU, U2 TLV74318PDBVR

Commit message: gerbers for production
Parts:
- U2: footprint Package_TO_SOT_SMD:SOT-23-5 -> bots:SOT-23-5
Connections:
- net GND: no longer H1.1, H2.1, H3.1, H4.1
