File: MidPlate/usb_pd.kicad_sch (KiCad schematic)
At the start: 22 parts, among them J9 USB_C_Receptacle_USB2.0_16P, Q5 PMOS, U4 HUSB238_xxxDD

Commit message: add adafruit connector
Parts:
- C9: footprint (none) -> Capacitor_SMD:CP_Elec_4x5.4
Changed lines of the file:
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@@
 			)
 		)
-		(property "Footprint" ""
+		(property "Footprint" "Capacitor_SMD:CP_Elec_4x5.4"
 			(at 123.19 92.71 0)
 			(hide yes)
@@
 			)
 		)
-		(property "Datasheet" ""
+		(property "Datasheet" "https://jlcpcb.com/partdetail/DMBJ-RVT1H1R0M0405_1UF50V/C970594"
 			(at 123.19 92.71 0)
 			(hide yes)
