File: MidPlate/imu.kicad_sch (KiCad schematic)
At the start: 1 part, among them U2 LSM6DSOX

Commit message: skidplate, then realized its pointless
Parts:
- U2: footprint bots:PQFN50P300X250X86-14N -> LSM6DSOX:PQFN50P250X300X86-14N
Changed lines of the file:
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@@
 			)
 		)
-		(property "Footprint" "bots:PQFN50P300X250X86-14N"
+		(property "Footprint" "LSM6DSOX:PQFN50P250X300X86-14N"
 			(at 132.08 85.09 0)
 			(hide yes)
